File: PCB/PCB.kicad_pcb (KiCad board)
At the start: 2 copper layers, 121.6 x 124.9 mm, 27 parts, among them J1 Conn_01x06, Q1 2N3904, U1 ATtiny85-20PU

Commit message: Changed default version to remove UNH logo
Parts:
- removed the G*** at (127.0, 81.3)
